Commit message: urdf updated

File: mirobot_description/urdf/mirobot_urdf_2.urdf (robot description, URDF)
Before this commit: robot mirobot, 7 links, 6 joints
Links:
- added link world
Joints:
- added joint joint_w: type fixed, parent world, child base_link

Commit message: ee added

File: mirobot_description/urdf/mirobot_urdf_2.urdf (robot description, URDF)
Before this commit: robot mirobot, 8 links, 7 joints
Links:
- added link ee_link; collision box size=0.01 0.01 0.01
Joints:
- added joint ee_fixed_joint: type fixed, parent Link6, child ee_link, origin xyz=0.0 0.0 0.0 rpy=0.0 1.5708 0.0
